Commit message: Make ghost red to distinguish it

File: packages/eyeinthesky/urdf/eyeinthesky_ghost.xacro (robot description, xacro)
@@ -92,3 +92,7 @@
     <gravity>false</gravity>
   </gazebo>
+  <!-- Special ghost colour! -->
+  <gazebo reference="chassis">
+    <material>Gazebo/Red</material>
+  </gazebo>
 </robot>
