Commit message: Add downward-facing camera to drone

File: packages/eyeinthesky/urdf/eyeinthesky.xacro (robot description, xacro)
@@ -1,95 +1,211 @@
 <?xml version='1.0'?>
 <robot name="robot" xmlns:xacro="http://www.ros.org/wiki/xacro">
-  <xacro:property name="camera_width" value="0.02"/>
-  <xacro:property name="camera_length" value="0.02"/>
-  <xacro:property name="camera_height" value="0.01"/>
-  <xacro:property name="camera_mass" value="0.01"/>
-  <xacro:property name="chassis_height" value="0.05"/>
-  <xacro:property name="chassis_mass" value="100000009.99"/>
-  <xacro:property name="chassis_radius" value="0.1"/>
-  <xacro:include filename="$(find robbie)/urdf/macros.xacro"/>
-  <!-- Body -->
-  <link name='chassis'>
-    <xacro:cylinder_inertial name="chassis" m="${chassis_mass}" r="${chassis_radius}" h="${chassis_height}"/>
-    <collision name='chassis_collision'>
+<xacro:property name="camera_width" value="0.02"/>
+<xacro:property name="camera_length" value="0.02"/>
+<xacro:property name="camera_height" value="0.01"/>
+<xacro:property name="camera_mass" value="0.01"/>
+<xacro:property name="chassis_height" value="0.05"/>
+<xacro:property name="chassis_mass" value="20"/>
+<xacro:property name="chassis_radius" value="0.1"/>
+<xacro:property name="leg_radius"  value="0.005"/>
+<xacro:property name="leg_length"  value="0.04"/>
+<xacro:property name="leg_mass"    value="0.05"/>
+<xacro:property name="down_cam_radius" value="0.01"/>
+<xacro:property name="down_cam_height" value="0.005"/>
+<xacro:property name="down_cam_mass"   value="0.01"/>
+<xacro:include filename="$(find robbie)/urdf/macros.xacro"/>
+<!-- Body -->
+<link name='chassis'>
+  <xacro:cylinder_inertial name="chassis" m="${chassis_mass}" r="${chassis_radius}" h="${chassis_height}"/>
+  <collision name='chassis_collision'>
+    <geometry>
+      <cylinder radius="${chassis_radius}" length="${chassis_height}"/>
+    </geometry>
+  </collision>
+  <visual name='chassis_visual'>
+    <origin xyz="0 0 0" rpy="0 0 0"/>
+    <geometry>
+      <cylinder radius="${chassis_radius}" length="${chassis_height}"/>
+    </geometry>
+  </visual>
+</link>
+<!-- Force Controller -->
+<gazebo>
+  <plugin name="chassis" filename="libgazebo_ros_force.so">
+    <bodyName>chassis</bodyName>
+    <topicName>/B1/cmd_force</topicName>
+  </plugin>
+</gazebo>
+<gazebo reference="chassis">
+  <enable_wind>true</enable_wind>
+</gazebo>
+<!-- Forward Camera -->
+<link name='camera_link'>
+  <xacro:box_inertial name="camera_link" m="${camera_mass}" x="${camera_width}" y="${camera_length}" z="${camera_height}"/>
+  <collision name='camera_link_collision'>
+    <geometry>
+      <box size="${camera_length} ${camera_width} ${camera_height}"/>
+    </geometry>
+  </collision>
+  <visual name='camera_link_visual'>
+    <origin xyz="0 0 0" rpy="0 0 0"/>
+    <geometry>
+      <box size="${camera_length} ${camera_width} ${camera_height}"/>
+    </geometry>
+  </visual>
+</link>
+<joint name="camera_joint" type="fixed">
+  <parent link="chassis"/>
+  <child link="camera_link"/>
+  <origin xyz="${chassis_radius} 0 ${chassis_height/2 - camera_height/2 - 0.0001}"/>
+</joint>
+<gazebo reference="camera_link">
+  <sensor type="camera" name="camera1">
+    <update_rate>30.0</update_rate>
+    <camera name="head">
+      <horizontal_fov>2.094395</horizontal_fov>
+      <image>
+        <width>800</width>
+        <height>800</height>
+        <format>R8G8B8</format>
+      </image>
+      <clip>
+        <near>0.02</near>
+        <far>300</far>
+      </clip>
+      <noise>
+        <type>gaussian</type>
+        <mean>0.0</mean>
+        <stddev>0.007</stddev>
+      </noise>
+    </camera>
+    <plugin name="camera_controller" filename="libgazebo_ros_camera.so">
+      <alwaysOn>true</alwaysOn>
+      <updateRate>0.0</updateRate>
+      <cameraName>rrbot/camera1</cameraName>
+      <imageTopicName>image_raw</imageTopicName>
+      <cameraInfoTopicName>camera_info</cameraInfoTopicName>
+      <frameName>camera_link</frameName>
+      <hackBaseline>0.07</hackBaseline>
+      <distortionK1>0.0</distortionK1>
+      <distortionK2>0.0</distortionK2>
+      <distortionK3>0.0</distortionK3>
+      <distortionT1>0.0</distortionT1>
+      <distortionT2>0.0</distortionT2>
+    </plugin>
+  </sensor>
+</gazebo>
+<!-- Downward Camera -->
+<link name='camera_down_link'>
+  <xacro:cylinder_inertial name="camera_down_link" m="${down_cam_mass}" r="${down_cam_radius}" h="${down_cam_height}"/>
+  <collision name='camera_down_link_collision'>
+    <geometry>
+      <cylinder radius="${down_cam_radius}" length="${down_cam_height}"/>
+    </geometry>
+  </collision>
+  <visual name='camera_down_link_visual'>
+    <origin xyz="0 0 0" rpy="0 0 0"/>
+    <geometry>
+      <cylinder radius="${down_cam_radius}" length="${down_cam_height}"/>
+    </geometry>
+  </visual>
+</link>
+<joint name="camera_down_joint" type="fixed">
+  <parent link="chassis"/>
+  <child link="camera_down_link"/>
+  <origin xyz="0 0 ${-(chassis_height/2) - (down_cam_height/2)}"
+          rpy="0 ${pi/2} 0"/>
+</joint>
+<gazebo reference="camera_down_link">
+  <sensor type="camera" name="camera_down">
+    <update_rate>30.0</update_rate>
+    <camera name="head">
+      <horizontal_fov>2.094395</horizontal_fov> <!--120 deg-->
+      <image>
+        <width>800</width>
+        <height>800</height>
+        <format>R8G8B8</format>
+      </image>
+      <clip>
+        <near>0.02</near>
+        <far>300</far>
+      </clip>
+      <noise>
+        <type>gaussian</type>
+        <mean>0.0</mean>
+        <stddev>0.007</stddev>
+      </noise>
+    </camera>
+    <plugin name="camera_down_controller" filename="libgazebo_ros_camera.so">
+      <alwaysOn>true</alwaysOn>
+      <updateRate>0.0</updateRate>
+      <cameraName>rrbot/camera_down</cameraName>
+      <imageTopicName>image_raw</imageTopicName>
+      <cameraInfoTopicName>camera_info</cameraInfoTopicName>
+      <frameName>camera_down_link</frameName>
+      <hackBaseline>0.07</hackBaseline>
+      <distortionK1>0.0</distortionK1>
+      <distortionK2>0.0</distortionK2>
+      <distortionK3>0.0</distortionK3>
+      <distortionT1>0.0</distortionT1>
+      <distortionT2>0.0</distortionT2>
+    </plugin>
+  </sensor>
+</gazebo>
+<!-- Legs -->
+<!-- Legs drop below chassis by leg_length*cos(tilt), camera needs clearance of down_cam_height -->
+<!-- leg_length=0.04 gives ~0.038m clearance at 20deg tilt, comfortably > down_cam_height=0.005m -->
+<xacro:macro name="landing_leg" params="name angle">
+  <link name="leg_${name}">
+    <xacro:cylinder_inertial name="leg_${name}" m="${leg_mass}" r="${leg_radius}" h="${leg_length}"/>
+    <collision name="leg_${name}_collision">
       <geometry>
-        <cylinder radius="${chassis_radius}" length="${chassis_height}"/>
+        <cylinder radius="${leg_radius}" length="${leg_length}"/>
       </geometry>
     </collision>
-    <visual name='chassis_visual'>
-      <origin xyz="0 0 0" rpy=" 0 0 0"/>
+    <visual name="leg_${name}_visual">
+      <origin xyz="0 0 0" rpy="0 0 0"/>
       <geometry>
-        <cylinder radius="${chassis_radius}" length="${chassis_height}"/>
+        <cylinder radius="${leg_radius}" length="${leg_length}"/>
       </geometry>
     </visual>
   </link>
-  <!-- Force Controller -->
-  <gazebo>
-    <plugin name="chassis" filename="libgazebo_ros_force.so">
-      <bodyName>chassis</bodyName>
-      <topicName>/D1/cmd_force</topicName>
-    </plugin>
-  </gazebo>
-  <gazebo reference="chassis">
-    <enable_wind>true</enable_wind>
-  </gazebo>
-  <!-- Camera -->
-  <link name='camera_link'>
-    <xacro:box_inertial name="camera_link" m="${camera_mass}" x="${camera_width}" y="${camera_length}" z="${camera_height}"/>
-    <collision name='camera_link_collision'>
-      <geometry>
-        <box size="${camera_length} ${camera_width} ${camera_height}"/>
-      </geometry>
-    </collision>
-    <visual name='camera_link_visual'>
-      <origin xyz="0 0 0" rpy=" 0 0 0"/>
-      <geometry>
-        <box size="${camera_length} ${camera_width} ${camera_height}"/>
-      </geometry>
-    </visual>
-  </link>
-  <joint name="camera_joint" type="fixed">
+  <!--
+    Place leg at chassis edge (chassis_radius - leg_radius) in XY, at the bottom face in Z.
+    rpy tilts the leg outward by 20deg around the axis tangent to the chassis edge,
+    so the foot splays out for stability while the top stays at the chassis rim.
+    The leg link origin is at its center, so offset by half leg_length downward.
+  -->
+  <joint name="leg_${name}_joint" type="fixed">
     <parent link="chassis"/>
-    <child link="camera_link"/>
-    <origin xyz="${chassis_radius} 0 ${chassis_height/2+camera_height/2}"/>
+    <child link="leg_${name}"/>
+    <origin xyz="${cos(radians(angle)) * (chassis_radius - leg_radius)}
+                 ${sin(radians(angle)) * (chassis_radius - leg_radius)}
+                 ${-(chassis_height/2) - (leg_length/2) * cos(0.349)}"
+            rpy="${sin(radians(angle)) * 0.349} ${-cos(radians(angle)) * 0.349} 0"/>
   </joint>
-  <gazebo reference="camera_link">
-    <sensor type="camera" name="camera1">
-      <update_rate>30.0</update_rate>
-      <camera name="head">
-        <horizontal_fov>2.094395</horizontal_fov> <!--120 deg-->
-        <image>
-          <width>800</width>
-          <height>800</height>
-          <format>R8G8B8</format>
-        </image>
-        <clip>
-          <near>0.02</near>
-          <far>300</far>
-        </clip>
-        <noise>
-          <type>gaussian</type>
-          <!-- Noise is sampled independently per pixel on each frame.
-              That pixel's noise value is added to each of its color
-              channels, which at that point lie in the range [0,1]. -->
-          <mean>0.0</mean>
-          <stddev>0.007</stddev>
-        </noise>
-      </camera>
-      <plugin name="camera_controller" filename="libgazebo_ros_camera.so">
-        <alwaysOn>true</alwaysOn>
-        <updateRate>0.0</updateRate>
-        <cameraName>rrbot/camera1</cameraName>
-        <imageTopicName>image_raw</imageTopicName>
-        <cameraInfoTopicName>camera_info</cameraInfoTopicName>
-        <frameName>camera_link</frameName>
-        <hackBaseline>0.07</hackBaseline>
-        <distortionK1>0.0</distortionK1>
-        <distortionK2>0.0</distortionK2>
-        <distortionK3>0.0</distortionK3>
-        <distortionT1>0.0</distortionT1>
-        <distortionT2>0.0</distortionT2>
-      </plugin>
-    </sensor>
-  </gazebo>
+</xacro:macro>
+<xacro:landing_leg name="front"  angle="0"/>
+<xacro:landing_leg name="left"   angle="90"/>
+<xacro:landing_leg name="back"   angle="180"/>
+<xacro:landing_leg name="right"  angle="270"/>
+<!-- Colours! -->
+<gazebo reference="camera_link">
+  <material>Gazebo/Purple</material>
+</gazebo>
+<gazebo reference="camera_down_link">
+  <material>Gazebo/Purple</material>
+</gazebo>
+<gazebo reference="leg_front">
+  <material>Gazebo/Black</material>
+</gazebo>
+<gazebo reference="leg_left">
+  <material>Gazebo/Black</material>
+</gazebo>
+<gazebo reference="leg_back">
+  <material>Gazebo/Black</material>
+</gazebo>
+<gazebo reference="leg_right">
+  <material>Gazebo/Black</material>
+</gazebo>
 </robot>

Commit message: Update drone to not exceed max weight of 20kg and use minimum mass for non-chassis joints

File: packages/eyeinthesky/urdf/eyeinthesky.xacro (robot description, xacro)
@@ -6,9 +6,9 @@
 <xacro:property name="camera_mass" value="0.01"/>
 <xacro:property name="chassis_height" value="0.05"/>
-<xacro:property name="chassis_mass" value="20"/>
+<xacro:property name="chassis_mass" value="19.94"/>
 <xacro:property name="chassis_radius" value="0.1"/>
 <xacro:property name="leg_radius"  value="0.005"/>
 <xacro:property name="leg_length"  value="0.04"/>
-<xacro:property name="leg_mass"    value="0.05"/>
+<xacro:property name="leg_mass"    value="0.01"/>
 <xacro:property name="down_cam_radius" value="0.01"/>
 <xacro:property name="down_cam_height" value="0.005"/>

Commit message: Add range sensors and liftoff mode

File: packages/eyeinthesky/urdf/eyeinthesky.xacro (robot description, xacro)
@@ -4,16 +4,17 @@
 <xacro:property name="camera_length" value="0.02"/>
 <xacro:property name="camera_height" value="0.01"/>
-<xacro:property name="camera_mass" value="0.01"/>
 <xacro:property name="chassis_height" value="0.05"/>
-<xacro:property name="chassis_mass" value="19.94"/>
 <xacro:property name="chassis_radius" value="0.1"/>
 <xacro:property name="leg_radius"  value="0.005"/>
 <xacro:property name="leg_length"  value="0.04"/>
-<xacro:property name="leg_mass"    value="0.01"/>
 <xacro:property name="down_cam_radius" value="0.01"/>
 <xacro:property name="down_cam_height" value="0.005"/>
-<xacro:property name="down_cam_mass"   value="0.01"/>
+<xacro:property name="range_size" value="0.01"/>
+<xacro:property name="camera_mass" value="0.01"/>
+<xacro:property name="down_cam_mass" value="0.01"/>
+<xacro:property name="leg_mass" value="0.01"/>
+<xacro:property name="range_mass" value="0.01"/>
+<xacro:property name="chassis_mass" value="19.91"/>
 <xacro:include filename="$(find robbie)/urdf/macros.xacro"/>
-<!-- Body -->
 <link name='chassis'>
   <xacro:cylinder_inertial name="chassis" m="${chassis_mass}" r="${chassis_radius}" h="${chassis_height}"/>
@@ -30,5 +31,4 @@
   </visual>
 </link>
-<!-- Force Controller -->
 <gazebo>
   <plugin name="chassis" filename="libgazebo_ros_force.so">
@@ -40,5 +40,14 @@
   <enable_wind>true</enable_wind>
 </gazebo>
-<!-- Forward Camera -->
+<gazebo>
+  <plugin name="imu_plugin" filename="libgazebo_ros_imu.so">
+    <alwaysOn>true</alwaysOn>
+    <bodyName>chassis</bodyName>
+    <topicName>imu/data</topicName>
+    <serviceName>imu/service</serviceName>
+    <gaussianNoise>0.0</gaussianNoise>
+    <updateRate>100.0</updateRate>
+  </plugin>
+</gazebo>
 <link name='camera_link'>
   <xacro:box_inertial name="camera_link" m="${camera_mass}" x="${camera_width}" y="${camera_length}" z="${camera_height}"/>
@@ -96,5 +105,4 @@
   </sensor>
 </gazebo>
-<!-- Downward Camera -->
 <link name='camera_down_link'>
   <xacro:cylinder_inertial name="camera_down_link" m="${down_cam_mass}" r="${down_cam_radius}" h="${down_cam_height}"/>
@@ -121,6 +129,5 @@
     <update_rate>30.0</update_rate>
     <camera name="head">
-      <horizontal_fov>2.094395</horizontal_fov> <!--120 deg-->
-      <image>
+      <horizontal_fov>2.094395</horizontal_fov> <image>
         <width>800</width>
         <height>800</height>
@@ -153,7 +160,65 @@
   </sensor>
 </gazebo>
-<!-- Legs -->
-<!-- Legs drop below chassis by leg_length*cos(tilt), camera needs clearance of down_cam_height -->
-<!-- leg_length=0.04 gives ~0.038m clearance at 20deg tilt, comfortably > down_cam_height=0.005m -->
+<xacro:macro name="range_sensor" params="name *origin">
+  <link name="${name}_link">
+    <xacro:box_inertial name="${name}_link" m="${range_mass}" x="${range_size}" y="${range_size}" z="${range_size}"/>
+    <collision name="${name}_collision">
+      <geometry>
+        <box size="${range_size} ${range_size} ${range_size}"/>
+      </geometry>
+    </collision>
+    <visual name="${name}_visual">
+      <geometry>
+        <box size="${range_size} ${range_size} ${range_size}"/>
+      </geometry>
+    </visual>
+  </link>
+  <joint name="${name}_joint" type="fixed">
+    <parent link="chassis"/>
+    <child link="${name}_link"/>
+    <xacro:insert_block name="origin" />
+  </joint>
+  <gazebo reference="${name}_link">
+    <sensor type="ray" name="${name}_sensor">
+      <pose>0 0 0 0 0 0</pose>
+      <visualize>true</visualize>
+      <update_rate>50</update_rate>
+      <ray>
+        <scan>
+          <horizontal>
+            <samples>10</samples>
+            <resolution>1</resolution>
+            <min_angle>-0.1</min_angle>
+            <max_angle>0.1</max_angle>
+          </horizontal>
+        </scan>
+        <range>
+          <min>0.05</min>
+          <max>10.0</max>
+          <resolution>0.01</resolution>
+        </range>
+      </ray>
+      <plugin filename="libgazebo_ros_range.so" name="${name}_plugin">
+        <gaussianNoise>0.005</gaussianNoise>
+        <alwaysOn>true</alwaysOn>
+        <updateRate>50</updateRate>
+        <topicName>range/${name}</topicName>
+        <frameName>${name}_link</frameName>
+        <radiation>INFRARED</radiation>
+        <fov>0.2</fov>
+      </plugin>
+    </sensor>
+    <material>Gazebo/Yellow</material>
+  </gazebo>
+</xacro:macro>
+<xacro:range_sensor name="range_left">
+  <origin xyz="0 ${chassis_radius} ${chassis_height/2 - camera_height/2 - 0.0001}" rpy="0 0 ${pi/2}"/>
+</xacro:range_sensor>
+<xacro:range_sensor name="range_backward">
+  <origin xyz="${-chassis_radius} 0 ${chassis_height/2 - camera_height/2 - 0.0001}" rpy="0 0 ${pi}"/>
+</xacro:range_sensor>
+<xacro:range_sensor name="range_down">
+  <origin xyz="${chassis_radius/2} 0 ${-(chassis_height/2) - (range_size/2)}" rpy="0 ${pi/2} 0"/>
+</xacro:range_sensor>
 <xacro:macro name="landing_leg" params="name angle">
   <link name="leg_${name}">
@@ -171,10 +236,4 @@
     </visual>
   </link>
-  <!--
-    Place leg at chassis edge (chassis_radius - leg_radius) in XY, at the bottom face in Z.
-    rpy tilts the leg outward by 20deg around the axis tangent to the chassis edge,
-    so the foot splays out for stability while the top stays at the chassis rim.
-    The leg link origin is at its center, so offset by half leg_length downward.
-  -->
   <joint name="leg_${name}_joint" type="fixed">
     <parent link="chassis"/>
@@ -190,5 +249,4 @@
 <xacro:landing_leg name="back"   angle="180"/>
 <xacro:landing_leg name="right"  angle="270"/>
-<!-- Colours! -->
 <gazebo reference="camera_link">
   <material>Gazebo/Purple</material>

Commit message: Remove extra sensors from drone

File: packages/eyeinthesky/urdf/eyeinthesky.xacro (robot description, xacro)
@@ -8,12 +8,12 @@
 <xacro:property name="leg_radius"  value="0.005"/>
 <xacro:property name="leg_length"  value="0.04"/>
-<xacro:property name="down_cam_radius" value="0.01"/>
-<xacro:property name="down_cam_height" value="0.005"/>
-<xacro:property name="range_size" value="0.01"/>
+<!-- <xacro:property name="down_cam_radius" value="0.01"/>
+<xacro:property name="down_cam_height" value="0.005"/> -->
+<!-- <xacro:property name="range_size" value="0.01"/> -->
 <xacro:property name="camera_mass" value="0.01"/>
-<xacro:property name="down_cam_mass" value="0.01"/>
+<!-- <xacro:property name="down_cam_mass" value="0.01"/> -->
 <xacro:property name="leg_mass" value="0.01"/>
-<xacro:property name="range_mass" value="0.01"/>
-<xacro:property name="chassis_mass" value="19.91"/>
+<!-- <xacro:property name="range_mass" value="0.01"/> -->
+<xacro:property name="chassis_mass" value="19.95"/>
 <xacro:include filename="$(find robbie)/urdf/macros.xacro"/>
 <link name='chassis'>
@@ -40,5 +40,5 @@
   <enable_wind>true</enable_wind>
 </gazebo>
-<gazebo>
+<!-- <gazebo>
   <plugin name="imu_plugin" filename="libgazebo_ros_imu.so">
     <alwaysOn>true</alwaysOn>
@@ -49,5 +49,5 @@
     <updateRate>100.0</updateRate>
   </plugin>
-</gazebo>
+</gazebo> -->
 <link name='camera_link'>
   <xacro:box_inertial name="camera_link" m="${camera_mass}" x="${camera_width}" y="${camera_length}" z="${camera_height}"/>
@@ -105,5 +105,5 @@
   </sensor>
 </gazebo>
-<link name='camera_down_link'>
+<!-- <link name='camera_down_link'>
   <xacro:cylinder_inertial name="camera_down_link" m="${down_cam_mass}" r="${down_cam_radius}" h="${down_cam_height}"/>
   <collision name='camera_down_link_collision'>
@@ -118,6 +118,6 @@
     </geometry>
   </visual>
-</link>
-<joint name="camera_down_joint" type="fixed">
+</link> -->
+<!-- <joint name="camera_down_joint" type="fixed">
   <parent link="chassis"/>
   <child link="camera_down_link"/>
@@ -159,6 +159,6 @@
     </plugin>
   </sensor>
-</gazebo>
-<xacro:macro name="range_sensor" params="name *origin">
+</gazebo> -->
+<!-- <xacro:macro name="range_sensor" params="name *origin">
   <link name="${name}_link">
     <xacro:box_inertial name="${name}_link" m="${range_mass}" x="${range_size}" y="${range_size}" z="${range_size}"/>
@@ -220,5 +220,5 @@
 <xacro:range_sensor name="range_down">
   <origin xyz="${chassis_radius/2} 0 ${-(chassis_height/2) - (range_size/2)}" rpy="0 ${pi/2} 0"/>
-</xacro:range_sensor>
+</xacro:range_sensor> -->
 <xacro:macro name="landing_leg" params="name angle">
   <link name="leg_${name}">
@@ -252,7 +252,7 @@
   <material>Gazebo/Purple</material>
 </gazebo>
-<gazebo reference="camera_down_link">
+<!-- <gazebo reference="camera_down_link">
   <material>Gazebo/Purple</material>
-</gazebo>
+</gazebo> -->
 <gazebo reference="leg_front">
   <material>Gazebo/Black</material>
